File: Hardware/Qwiic_PT100.brd (EAGLE design)
At the start: 38.1 x 38.1 mm, 85 parts, among them IC1 ADS122C04IPWR, J2 QWIIC_RIGHT_ANGLE, J3 PTH, J4 QWIIC_RIGHT_ANGLE

Commit message: Tweaks
Parts:
- added TP1, TP2, TP3, TP4: TEST-POINTTP_15TH_THRU, SparkFun-Connectors:TP_15TH
- added U$21: (no value), 4_small:40
- added U$27: (no value), buzzard_labels (5):31
- added U$28: (no value), buzzard_labels (5):20
- added U$35: (no value), buzzard_labels (5):15
- moved J3 1.27 mm to (17.8, 1.27)
- moved J5 1.27 mm to (15.2, 1.27)
- moved J6 1.27 mm to (12.7, 1.27)
- moved U$10 1.27 mm to (22.9, 6.35)
- moved U$14 1.27 mm to (12.7, 6.99)
- moved U$15 1.27 mm to (12.7, 1.65)
- moved U$16 1.27 mm to (15.2, 7.37)
- moved U$17 1.27 mm to (15.2, 1.40)
- moved U$23 1.27 mm to (25.4, 1.78)
- moved U$24 1.27 mm to (22.9, 1.65)
- moved U$25 1.27 mm to (17.8, 1.65)
- moved U$26 1.27 mm to (20.3, 1.78)
- moved U$3 1.27 mm to (20.3, 6.48)
- moved U$7 1.27 mm to (17.8, 6.48)
- moved U$9 1.27 mm to (25.4, 6.22)
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Connections:
- net AIN3: now also TP1.P$1
- net N$1: now also TP2.P$1
- net N$5: now also TP3.P$1
- net N$6: now also TP4.P$1
Routing:
- net GND: track 35.3 -> 37.3 mm
- net AIN3: track 24.9 -> 26.8 mm
- net N$1: track 19.3 -> 21.1 mm
- net N$5: track 18.6 -> 20.4 mm
- net N$6: track 24.1 -> 25.8 mm
- net !RESET: track 20.7 -> 22.1 mm
- net !DRDY: track 27.5 -> 28.2 mm
- net A1: track 7.18 -> 6.50 mm
- net SCL: track 72.7 -> 73.3 mm
